File: eagle/c65Keyb.brd (EAGLE design)
At the start: 93 x 160 mm, 94 parts, among them Q1 8Mhz, U1 STM32F407IET6__FI__, U2 744245, U3 744245, U4 744245, X4 MKDS_5/3-6,35

Commit message: added LED support and updated the eagle schematics
Parts:
- C21, C22: value 100nF -> 33pF
Changed lines of the file:
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@@
 <?xml version="1.0" encoding="utf-8"?>
 <!DOCTYPE eagle SYSTEM "eagle.dtd">
-<eagle version="7.2.0">
+<eagle version="7.1.0">
 <drawing>
 <settings>
@@
 <attribute name="VALUE" x="36.83" y="85.725" size="1.27" layer="27" rot="R270"/>
 </element>
-<element name="C21" library="rcl" package="C0805" value="100nF" x="43.97375" y="92.3925" smashed="yes" rot="R180">
+<element name="C21" library="rcl" package="C0805" value="33pF" x="43.97375" y="92.3925" smashed="yes" rot="R180">
 <attribute name="NAME" x="45.24375" y="91.1225" size="1.27" layer="25" rot="R180"/>
 <attribute name="VALUE" x="45.24375" y="94.9325" size="1.27" layer="27" rot="R180"/>
 </element>
-<element name="C22" library="rcl" package="C0805" value="100nF" x="37.30625" y="92.3925" smashed="yes">
+<element name="C22" library="rcl" package="C0805" value="33pF" x="37.30625" y="92.3925" smashed="yes">
 <attribute name="NAME" x="38.89375" y="91.1225" size="1.27" layer="25" rot="R180"/>
 <attribute name="VALUE" x="36.03625" y="89.8525" size="1.27" layer="27"/>
